File: static-fmreceiver.kicad_pcb (KiCad board)
At the start: 2 copper layers, 67.9 x 43.8 mm, 20 parts, among them J1 Conn_01x02 (SPKR_R), J2 Conn_01x02 (SPKR_L), SW1 SW_Push, SW2 SW_Push, U1 RDA5807MRRD-102V2.0, U2 XIAO-RP2040-DIP, U3 TDA2822NBD

Commit message: done with pcb methink
lots of silkscreen and optimised routing. I think it looks kinda nice
Parts:
- added CN1: PJ-3200, Static:AUDIO-TH_PJ-3200, F.Cu at (186.6, 57.0)
- added G***: LOGO, LOGO, F.Cu at (170.4, 77.1)
- added G***: LOGO, LOGO, B.Cu at (189.3, 72.2)
- added G***: LOGO, LOGO, B.Cu at (151.8, 72.1)
- added G***: LOGO, LOGO, B.Cu at (172.3, 60.3)
- added G***: LOGO, LOGO, F.Cu at (191.2, 47.7)
- added G***: LOGO, LOGO, F.Cu at (221.4, 66.6)
- added G***: LOGO, LOGO, F.Cu at (146.1, 86.0)
- added G***: LOGO, LOGO, F.Cu at (205.6, 40.9)
- added G***: LOGO, LOGO, F.Cu at (176.4, 35.7)
- added G***: LOGO, LOGO, F.Cu at (146.5, 44.7)
- added G***: LOGO, LOGO, F.Cu at (191.1, 88.0)
- added G***: LOGO, LOGO, B.Cu at (163.7, 71.7)
- C5 470uF: renamed from C5
- SW2: footprint Button_Switch_Keyboard:SW_Cherry_MX_1.00u_PCB -> Connector_PinHeader_2.54mm:PinHeader_1x02_P2.54mm_Vertical
- moved SW2 75.4 mm to (180.9, 51.4), turned to 90 degrees
- moved C3 32.9 mm to (168.5, 83.4), turned to 0 degrees
- moved C5 470uF 31.2 mm to (163.8, 83.4)
- moved C1 28.6 mm to (154.8, 82.2), turned to 90 degrees
- moved SPK2 26.2 mm to (157.3, 86.7), turned to -90 degrees
- moved H3 19.1 mm to (148.5, 85.5)
- moved H1 18.7 mm to (148.5, 50.1)
- moved C4 13.3 mm to (149.3, 62.7), turned to 0 degrees
- moved RV2 11.9 mm to (162.8, 57.1)
- moved R1 11.6 mm to (158.1, 50.3)
- moved C2 8.63 mm to (156.5, 62.7)
- moved R2 8.63 mm to (167.2, 57.9)
- moved U3 8.40 mm to (148.5, 67.8)
- moved RV1 8.37 mm to (171.9, 57.2)
- moved U1 7.20 mm to (165.1, 71.5), turned to 90 degrees
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- renumbered J1 to SPK1, J2 to SPK2
Connections:
- SW2 pad 1: unconnected-(SW2-Pad1) -> GND
- SW2 pad 2: GND -> Net-(U2-P26_A0_D0)
- U2 pad 1: unconnected-(U2-P26_A0_D0-Pad1) -> Net-(U2-P26_A0_D0)
Routing:
- net Net-(U1-ANT): track 0.00 -> 29.4 mm
- net GND: track 23.6 -> 52.4 mm
- net /R_OUT: track 32.7 -> 10.2 mm
- net Net-(U2-P26_A0_D0): track 0.00 -> 15.9 mm
- net Net-(U3-OUT2): track 5.65 -> 19.6 mm
- net Net-(U3-IN2): track 44.2 -> 30.7 mm
- net /L_OUT: track 0.00 -> 10.8 mm
- net Net-(U3-OUT1): track 14.9 -> 5.87 mm
- net /SCL: track 27.7 -> 20.8 mm
- net Net-(U3-IN1): track 24.1 -> 29.1 mm
- net Net-(U2-P1_D7_RX): track 6.65 -> 10.3 mm
- net +3V3: track 61.3 -> 64.7 mm
- net /SDA: track 32.0 -> 29.9 mm
- net Net-(U3-NF2): track 15.0 -> 16.9 mm
- net Net-(U3-NF1): track 7.25 -> 5.80 mm
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Other:
- board size 67.9 x 43.8 mm -> 48.6 x 43.8 mm
- board text added: "Canberra On TOP"
- board text added: "HAVEN CANBERRA"
- board text added: "Henry Wauzivuff"
- board text added: "ingo.au"
- board text added: "southbag.cc"
