File: static-fmreceiver.kicad_sch (KiCad schematic)
At the start: 0 parts

Commit message: finish schematic probably  + readme
Parts:
- added C1, C2, C3: 100uF, Capacitor_THT:CP_Radial_D6.3mm_P2.50mm, symbol Device:C_Polarized
- added C4, C5: 470uF, Capacitor_THT:CP_Radial_D6.3mm_P2.50mm, symbol Device:C_Polarized
- added CN1: PJ-3200, easyeda2kicad:AUDIO-TH_PJ-3200, symbol Static_Symbol_Library:PJ-3200
- added H1, H2, H3, H4: MountingHole, MountingHole:MountingHole_2.7mm_M2.5, symbol Mechanical:MountingHole
- added J1: Conn_01x02 (SPKR_R), Connector_PinHeader_2.54mm:PinHeader_1x02_P2.54mm_Vertical, symbol Connector_Generic:Conn_01x02
- added J2: Conn_01x02 (SPKR_L), Connector_PinHeader_2.54mm:PinHeader_1x02_P2.54mm_Vertical, symbol Connector_Generic:Conn_01x02
- added R1, R2: 10K, Resistor_THT:R_Axial_DIN0207_L6.3mm_D2.5mm_P7.62mm_Horizontal, symbol Device:R
- added RV1, RV2: R_Potentiometer 10K, Connector_PinHeader_2.54mm:PinHeader_1x03_P2.54mm_Vertical, symbol Device:R_Potentiometer
- added SW1: SW_Push, Connector_PinHeader_2.54mm:PinHeader_1x02_P2.54mm_Vertical, symbol Switch:SW_Push
- added SW2: SW_Push, Button_Switch_Keyboard:SW_Cherry_MX_1.00u_PCB, symbol Switch:SW_Push
- added U1: RDA5807MRRD-102V2.0, Static:RDA5807, symbol Static_Symbol_Library:RDA5807MRRD-102V2.0
- added U2: XIAO-RP2040-DIP, Static:XIAO-RP2040-DIP, symbol Static_Symbol_Library:XIAO-RP2040-DIP
- added U3: TDA2822NBD, Package_DIP:DIP-8_W7.62mm, symbol Static_Symbol_Library:TDA2822NBD
Connections:
- new net: CN1.4, U1.10 (ANT)
- new net: R1.1, RV2.2, U3.6 (IN2)
- new net: SW1.1, U2.8 (P1_D7_RX)
- new net: C2.1, U3.8 (NF1)
- new net: R2.1, RV1.2, U3.7 (IN1)
- new net: C4.1, U3.1 (OUT1)
- new net: C5.1, U3.3 (OUT2)
- new net: C3.1, U3.5 (NF2)
- new net +3V3: C1.1, U1.5 (VCC), U2.12 (3V3), U3.2 (VCC)
- new net GND: C1.2, C2.2, C3.2, CN1.3, J1.2 (Pin_2), J2.2 (Pin_2), R1.2, R2.2, RV1.3, RV2.3, SW1.2, SW2.2, U1.3 (GND), U1.6 (GND), U1.9 (GND), U2.13 (GND), U3.4 (GND)
- new net L_AMP_OUT: C5.2, J2.1 (Pin_1)
- new net L_OUT: RV1.1, U1.7 (L-OUT)
- new net R_AMP_OUT: C4.2, J1.1 (Pin_1)
- new net R_OUT: RV2.1, U1.8 (R-OUT)
- new net SCL: U1.2 (CLK), U2.6 (P7_SCL_D5)
- new net SDA: U1.1 (DATA), U2.5 (P6_SDA_D4)
- no-connect marks 0 -> 10

Commit message: done with pcb methink
lots of silkscreen and optimised routing. I think it looks kinda nice
Parts:
- CN1: footprint easyeda2kicad:AUDIO-TH_PJ-3200 -> Static:AUDIO-TH_PJ-3200
- SW2: footprint Button_Switch_Keyboard:SW_Cherry_MX_1.00u_PCB -> Connector_PinHeader_2.54mm:PinHeader_1x02_P2.54mm_Vertical
Connections:
- net GND: now also SW2.1; no longer SW2.2
- net at U2.1 (P26_A0_D0): now also SW2.2
- no-connect marks 10 -> 9
Other:
- note added: "Audio Amps"
- note added: "Audio IC"
- note added: "Potentiometers"
- note added: "Radio IC"
- note added: "Speakers"
- note added: "Xiao"
- moved on the sheet: CN1, H1, H2, H3, H4, SW1, SW2, U1, U2
